File: PCB Design/ESP12E Brain.brd (EAGLE design)
At the start: 95.2 x 79.7 mm, 52 parts, among them IC1 LM1117T-1.8, T1 2N2222, T2 2N2222, T3 2N2222, T4 2N2222, X5 TB 3.5MM

Commit message: Updated brd file
Parts:
- removed IC1: LM1117T-1.8, lm1117:TO220
- added IC2: LM1117MPX-3.3, lm1117:SOT223
Connections:
- net +3V3: now also IC2.2; no longer IC1.2
- net +5V: now also IC2.3; no longer IC1.3
- net GND: now also IC2.1; no longer IC1.1
Routing:
- net +5V: track 259.0 -> 275.0 mm
- net +3V3: track 46.0 -> 50.7 mm, vias 0 -> 1
- net GND: track 233.9 -> 237.9 mm
