File: PCB Design/ESP12E Brain.sch (EAGLE design)
At the start: 52 parts, among them IC1 LM1117T-1.8, T1 2N2222, T2 2N2222, T3 2N2222, T4 2N2222, X5 TB 3.5MM

Commit message: Updated brd file
Parts:
- removed IC1: LM1117T-1.8, lm1117:LM1117T-1.8
- added IC2: LM1117MPX-3.3, lm1117:LM1117MPX-3.3
Connections:
- net +3V3: now also IC2.OUT; no longer IC1.OUT
- net +5V: now also IC2.IN; no longer IC1.IN
- net GND: now also IC2.GND; no longer IC1.GND
Changed lines of the file:
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@@
 <part name="P+12" library="supply1" library_urn="urn:adsk.eagle:library:371" deviceset="+5V" device=""/>
 <part name="R14" library="rcl" library_urn="urn:adsk.eagle:library:334" deviceset="R-EU_" device="0204/7" package3d_urn="urn:adsk.eagle:package:23498/2" value="220E"/>
-<part name="IC1" library="lm1117" deviceset="LM1117T-*" device="" technology="1.8"/>
 <part name="PROG" library="con-headers-jp" deviceset="M-1X04-" device="SIP-100-32" value="Male header"/>
 <part name="I2C" library="con-headers-jp" deviceset="M-1X04-" device="SIP-100-32" value="Male Header"/>
@@
 <part name="REL4" library="Rembrandt Electronics - Terminal Block 3-5mm v1-0" deviceset="TERMINAL-BLOCK-3.5MM-3-PIN" device="-ROUND-PAD" value="TB 3.5MM"/>
 <part name="X5" library="Rembrandt Electronics - Terminal Block 3-5mm v1-0" deviceset="TERMINAL-BLOCK-3.5MM-2-PIN" device="-ROUND-PAD" value="TB 3.5MM"/>
+<part name="IC2" library="lm1117" deviceset="LM1117MPX-*" device="" technology="3.3"/>
 </parts>
 <sheets>
@@
 <attribute name="VALUE" x="54.61" y="-18.542" size="1.778" layer="96"/>
 </instance>
-<instance part="IC1" gate="G$1" x="-48.26" y="76.2" smashed="yes">
-<attribute name="NAME" x="-45.72" y="68.58" size="1.778" layer="95"/>
-<attribute name="VALUE" x="-45.72" y="66.04" size="1.778" layer="96"/>
-</instance>
 <instance part="PROG" gate="G$1" x="-71.12" y="38.1" smashed="yes">
 <attribute name="VALUE" x="-74.93" y="27.94" size="1.778" layer="96"/>
@@
 <attribute name="NAME" x="-110.49" y="72.771" size="1.778" layer="95"/>
 <attribute name="VALUE" x="-97.79" y="72.771" size="1.778" layer="96"/>
+</instance>
+<instance part="IC2" gate="G$1" x="-48.26" y="76.2" smashed="yes">
+<attribute name="NAME" x="-45.72" y="68.58" size="1.778" layer="95"/>
+<attribute name="VALUE" x="-45.72" y="66.04" size="1.778" layer="96"/>
 </instance>
 </instances>
@@
 <pinref part="C2" gate="G$1" pin="-"/>
 <wire x1="-48.26" y1="63.5" x2="-38.1" y2="63.5" width="0.1524" layer="91"/>
-<pinref part="IC1" gate="G$1" pin="GND"/>
+<pinref part="IC2" gate="G$1" pin="GND"/>
+<junction x="-48.26" y="68.58"/>
 </segment>
 <segment>
@@
 <wire x1="-38.1" y1="71.12" x2="-38.1" y2="76.2" width="0.1524" layer="91"/>
 <junction x="-38.1" y="76.2"/>
-<pinref part="IC1" gate="G$1" pin="OUT"/>
+<pinref part="IC2" gate="G$1" pin="OUT"/>
 </segment>
 </net>
@@
 </segment>
 <segment>
-<wire x1="-60.96" y1="76.2" x2="-55.88" y2="76.2" width="0.1524" layer="91"/>
+<wire x1="-63.5" y1="76.2" x2="-55.88" y2="76.2" width="0.1524" layer="91"/>
 <pinref part="P+5" gate="1" pin="+5V"/>
 <wire x1="-71.12" y1="76.2" x2="-63.5" y2="76.2" width="0.1524" layer="91"/>
 <pinref part="C1" gate="G$1" pin="+"/>
-<wire x1="-63.5" y1="76.2" x2="-60.96" y2="76.2" width="0.1524" layer="91"/>
 <wire x1="-63.5" y1="71.12" x2="-63.5" y2="76.2" width="0.1524" layer="91"/>
 <junction x="-63.5" y="76.2"/>
-<pinref part="IC1" gate="G$1" pin="IN"/>
+<pinref part="IC2" gate="G$1" pin="IN"/>
 <junction x="-55.88" y="76.2"/>
 </segment>
